Commit message: Change parent_link and origin

File: robucar_description/urdf/robucar.xacro (robot description, xacro)
@@ -66,14 +66,14 @@
     </joint>
     <!-- Wheel macros -->
-    <xacro:jaguar_wheel_steered wheel_prefix="front_left">
+    <xacro:jaguar_wheel_steered wheel_prefix="front_left" parent_link="base_link">
       <origin xyz="${wheelbase/2+wheel_x_offset} ${track/2} ${wheel_vertical_offset}" rpy="0 0 0" />
     </xacro:jaguar_wheel_steered>
-    <xacro:jaguar_wheel_steered wheel_prefix="front_right">
+    <xacro:jaguar_wheel_steered wheel_prefix="front_right" parent_link="base_link">
       <origin xyz="${wheelbase/2+wheel_x_offset} ${-track/2} ${wheel_vertical_offset}" rpy="0 0 0" />
     </xacro:jaguar_wheel_steered>
-    <xacro:jaguar_wheel_steered wheel_prefix="rear_left">
+    <xacro:jaguar_wheel_steered wheel_prefix="rear_left" parent_link="base_link">
       <origin xyz="${-wheelbase/2+wheel_x_offset} ${track/2} ${wheel_vertical_offset}" rpy="0 0 0" />
     </xacro:jaguar_wheel_steered>
-    <xacro:jaguar_wheel_steered wheel_prefix="rear_right">
+    <xacro:jaguar_wheel_steered wheel_prefix="rear_right" parent_link="base_link">
       <origin xyz="${-wheelbase/2+wheel_x_offset} ${-track/2} ${wheel_vertical_offset}" rpy="0 0 0" />
     </xacro:jaguar_wheel_steered>

File: robucar_description/urdf/wheel_steered.xacro (robot description, xacro)
@@ -2,7 +2,7 @@
 <robot xmlns:xacro="http://ros.org/wiki/xacro" name="jaguar_wheel_steered">
   <xacro:include filename="$(find robucar_description)/urdf/wheel.xacro" />
-  <xacro:macro name="jaguar_wheel_steered" params="wheel_prefix *joint_pose">
-    <xacro:jaguar_wheel wheel_prefix="${wheel_prefix}">
-      <xacro:insert_block name="joint_pose"/>
+  <xacro:macro name="jaguar_wheel_steered" params="wheel_prefix parent_link *joint_origin">
+    <xacro:jaguar_wheel wheel_prefix="${wheel_prefix}" parent_link="${wheel_prefix}_steering">
+      <origin xyz="0 0 0" rpy="0 0 0" />
     </xacro:jaguar_wheel>
     <link name="${wheel_prefix}_steering"/>
@@ -10,7 +10,7 @@
       <limit lower="-1.57075" upper="1.57075" effort="-1" velocity="-1"/>
       <axis xyz="0 0 1"/>
-      <parent link="base_link"/>
+      <parent link="${parent_link}"/>
       <child link="${wheel_prefix}_steering"/>
-      <xacro:insert_block name="joint_pose"/>
+      <xacro:insert_block name="joint_origin"/>
     </joint>
   </xacro:macro>
