Commit message: Remove jaguar prefix from robucar description

File: robucar_description/urdf/description.xacro (robot description, xacro)
@@ -3,5 +3,5 @@
   <xacro:arg name="camera_enabled" default="false" />
   <xacro:arg name="navsat_enabled" default="true" />
-  <xacro:include filename="$(find robucar_description)/urdf/robucar.xacro" />
+  <xacro:include filename="$(find robucar_description)/urdf/robucar.urdf.xacro" />
   <xacro:robucar />
 </robot>

File: robucar_description/urdf/robucar.urdf.xacro (robot description, xacro)
@@ -3,5 +3,5 @@
   <xacro:arg name="laser_enabled" default="false" />
   <xacro:arg name="camera_enabled" default="false" />
-  <xacro:arg name="navsat_enabled" default="true" />
+  <xacro:arg name="navsat_enabled" default="false" />
   <xacro:include filename="$(find robucar_description)/urdf/wheel_steered.xacro" />
   <xacro:property name="M_PI" value="3.14159"/>
@@ -66,16 +66,16 @@
     </joint>
     <!-- Wheel macros -->
-    <xacro:jaguar_wheel_steered wheel_prefix="front_left" parent_link="base_link">
+    <xacro:wheel_steered wheel_prefix="front_left" parent_link="base_link">
       <origin xyz="${wheelbase/2+wheel_x_offset} ${track/2} ${wheel_vertical_offset}" rpy="0 0 0" />
-    </xacro:jaguar_wheel_steered>
-    <xacro:jaguar_wheel_steered wheel_prefix="front_right" parent_link="base_link">
+    </xacro:wheel_steered>
+    <xacro:wheel_steered wheel_prefix="front_right" parent_link="base_link">
       <origin xyz="${wheelbase/2+wheel_x_offset} ${-track/2} ${wheel_vertical_offset}" rpy="0 0 0" />
-    </xacro:jaguar_wheel_steered>
-    <xacro:jaguar_wheel_steered wheel_prefix="rear_left" parent_link="base_link">
+    </xacro:wheel_steered>
+    <xacro:wheel_steered wheel_prefix="rear_left" parent_link="base_link">
       <origin xyz="${-wheelbase/2+wheel_x_offset} ${track/2} ${wheel_vertical_offset}" rpy="0 0 0" />
-    </xacro:jaguar_wheel_steered>
-    <xacro:jaguar_wheel_steered wheel_prefix="rear_right" parent_link="base_link">
+    </xacro:wheel_steered>
+    <xacro:wheel_steered wheel_prefix="rear_right" parent_link="base_link">
       <origin xyz="${-wheelbase/2+wheel_x_offset} ${-track/2} ${wheel_vertical_offset}" rpy="0 0 0" />
-    </xacro:jaguar_wheel_steered>
+    </xacro:wheel_steered>
     <xacro:if value="$(arg laser_enabled)">
       <!-- Hokuyo UTM-30LX mounted upside down below the body -->

File: robucar_description/urdf/wheel.xacro (robot description, xacro)
@@ -1,8 +1,8 @@
 <?xml version="1.0"?>
-<robot xmlns:xacro="http://ros.org/wiki/xacro" name="jaguar_wheel">
+<robot xmlns:xacro="http://ros.org/wiki/xacro" name="wheel">
   <!--<xacro:property name="M_PI" default="3.14159"/>
   <xacro:property name="wheel_length" default="0.09" />
   <xacro:property name="wheel_radius" default="0.13" />-->
-  <xacro:macro name="jaguar_wheel" params="wheel_prefix parent_link *joint_origin">
+  <xacro:macro name="wheel" params="wheel_prefix parent_link *joint_origin">
     <gazebo reference="${wheel_prefix}_wheel_link">
       <material>Gazebo/Black</material>

File: robucar_description/urdf/wheel_steered.xacro (robot description, xacro)
@@ -1,9 +1,9 @@
 <?xml version="1.0"?>
-<robot xmlns:xacro="http://ros.org/wiki/xacro" name="jaguar_wheel_steered">
+<robot xmlns:xacro="http://ros.org/wiki/xacro" name="wheel_steered">
   <xacro:include filename="$(find robucar_description)/urdf/wheel.xacro" />
-  <xacro:macro name="jaguar_wheel_steered" params="wheel_prefix parent_link *joint_origin">
-    <xacro:jaguar_wheel wheel_prefix="${wheel_prefix}" parent_link="${wheel_prefix}_steering">
+  <xacro:macro name="wheel_steered" params="wheel_prefix parent_link *joint_origin">
+    <xacro:wheel wheel_prefix="${wheel_prefix}" parent_link="${wheel_prefix}_steering">
       <origin xyz="0 0 0" rpy="0 0 0" />
-    </xacro:jaguar_wheel>
+    </xacro:wheel>
     <link name="${wheel_prefix}_steering"/>
     <joint name="${wheel_prefix}_steering_joint" type="revolute">

Commit message: Add the velodyne on robucar

File: robucar_description/urdf/description.xacro (robot description, xacro)
@@ -3,4 +3,5 @@
   <xacro:arg name="camera_enabled" default="false" />
   <xacro:arg name="navsat_enabled" default="true" />
+  <xacro:arg name="velodyne_enabled" default="true" />
   <xacro:include filename="$(find robucar_description)/urdf/robucar.urdf.xacro" />
   <xacro:robucar />

File: robucar_description/urdf/robucar.urdf.xacro (robot description, xacro)
@@ -4,4 +4,5 @@
   <xacro:arg name="camera_enabled" default="false" />
   <xacro:arg name="navsat_enabled" default="false" />
+  <xacro:arg name="velodyne_enabled" default="false" />
   <xacro:include filename="$(find robucar_description)/urdf/wheel_steered.xacro" />
   <xacro:property name="M_PI" value="3.14159"/>
@@ -120,4 +121,10 @@
       </joint>
     </xacro:if>
+    <xacro:if value="$(arg velodyne_enabled)">
+    <xacro:include filename="$(find velodyne_description)/urdf/HDL-32E.urdf.xacro"/>
+    <HDL-32E parent="base_link" name="velodyne2" topic="/velodyne_points2">
+      <origin xyz="0 0 0.6" rpy="0 0 0" />
+    </HDL-32E>
+    </xacro:if>
   </xacro:macro>
 </robot>

File: robucar_gazebo/urdf/description.gazebo.xacro (robot description, xacro)
@@ -4,4 +4,5 @@
   <xacro:arg name="camera_enabled" default="false" />
   <xacro:arg name="navsat_enabled" default="false" />
+  <xacro:arg name="velodyne_enabled" default="false" />
   <xacro:include filename="$(find robucar_description)/urdf/robucar.urdf.xacro" />
   <xacro:include filename="$(find robucar_gazebo)/urdf/robucar.gazebo.xacro" />
