Commit message: [description] Use lighter meshes files

File: robucar_description/urdf/chassis.xacro (robot description, xacro)
@@ -20,5 +20,5 @@
         <geometry>
           <!--<box size="${base_x_size} ${base_y_size} ${base_z_size}"/>-->
-          <mesh filename="package://robucar_description/meshes/robufast_frame_0_72.dae"/>
+          <mesh filename="package://robucar_description/meshes/robufast_frame.dae"/>
         </geometry>
         <material name="grey">

File: robucar_description/urdf/wheel.xacro (robot description, xacro)
@@ -25,5 +25,5 @@
 				<geometry>
           <!--<cylinder length="${wheel_length}" radius="${wheel_radius}"/>-->
-          <mesh filename="package://robucar_description/meshes/robufast_wheel_d0_56.dae"/>
+          <mesh filename="package://robucar_description/meshes/robufast_wheel.dae"/>
 				</geometry>
         <material name="black">

Commit message: [description] change link position

File: robucar_description/urdf/chassis.xacro (robot description, xacro)
@@ -8,4 +8,11 @@
   <xacro:property name="wheelbase" value="1.22" />
   <xacro:property name="track" value="1.23" />
+  <!-- Wheel Mounting Positions -->
+  <xacro:property name="ground_clearance" value="0.19" />
+  <xacro:property name="wheel_x_offset" value="0.0" />
+  <xacro:property name="wheel_y_offset" value="0.1" />
+  <!-- LIDAR Properties -->
+  <xacro:property name="lidar_ground_clearance" value="0.69" />
+  <xacro:property name="lidar_x_offset" value="0.4" />
   <xacro:macro name="chassis">
     <!-- Base footprint is on the ground under the robot -->

File: robucar_description/urdf/robucar.urdf.xacro (robot description, xacro)
@@ -7,11 +7,4 @@
   <xacro:include filename="$(find robucar_description)/urdf/chassis.xacro" />
   <xacro:property name="M_PI" value="3.14159"/>
-  <!-- Wheel Mounting Positions -->
-  <xacro:property name="ground_clearance" value="0.19" />
-  <xacro:property name="wheel_x_offset" value="0.0" />
-  <xacro:property name="wheel_y_offset" value="0.05" />
-  <!-- LIDAR Properties -->
-  <xacro:property name="lidar_ground_clearance" value="0.69" />
-  <xacro:property name="lidar_x_offset" value="0.4" />
   <xacro:macro name="robucar">
     <xacro:chassis/>

File: robucar_description/urdf/robucar_4ws.urdf.xacro (robot description, xacro)
@@ -7,11 +7,4 @@
   <xacro:include filename="$(find robucar_description)/urdf/chassis.xacro" />
   <xacro:property name="M_PI" value="3.14159"/>
-  <!-- Wheel Mounting Positions -->
-  <xacro:property name="ground_clearance" value="0.19" />
-  <xacro:property name="wheel_x_offset" value="0.0" />
-  <xacro:property name="wheel_y_offset" value="0.05" />
-  <!-- LIDAR Properties -->
-  <xacro:property name="lidar_ground_clearance" value="0.69" />
-  <xacro:property name="lidar_x_offset" value="0.4" />
   <xacro:macro name="robucar">
     <xacro:chassis/>

File: robucar_description/urdf/wheel_steered.xacro (robot description, xacro)
@@ -8,5 +8,5 @@
     <link name="${wheel_prefix}_steering">
       <visual>
-        <origin xyz="0 ${-wheel_origin_y} 0" rpy="0 0 0"/>
+        <origin xyz="0 0 0" rpy="0 0 0"/>
         <geometry>
           <box size="0.05 ${steering_link_y} 0.05"/>
@@ -18,5 +18,5 @@
       <inertial>
         <mass value="${steering_link_mass}" />
-        <origin xyz="0 ${-wheel_origin_y} 0" />
+        <origin xyz="0 0 0" />
         <!--<inertia ixx="1.0" ixy="0" ixz="0"
                  iyy="1.0" iyz="0"

Commit message: Working parameters with false mass

File: robucar_description/urdf/chassis.xacro (robot description, xacro)
@@ -2,5 +2,5 @@
 <robot xmlns:xacro="http://www.ros.org/wiki/xacro" name="chassis">
   <!-- Base Properties -->
-  <xacro:property name="mass_base" value="340" />
+  <xacro:property name="mass_base" value="10" />
   <xacro:property name="base_x_size" value="1.66000" />
   <xacro:property name="base_y_size" value="0.60000" />
@@ -11,5 +11,5 @@
   <xacro:property name="ground_clearance" value="0.19" />
   <xacro:property name="wheel_x_offset" value="0.0" />
-  <xacro:property name="wheel_y_offset" value="0.1" />
+  <xacro:property name="wheel_y_offset" value="0.0" />
   <!-- LIDAR Properties -->
   <xacro:property name="lidar_ground_clearance" value="0.69" />
@@ -47,9 +47,9 @@
     <link name="inertial_link">
       <inertial>
-        <mass value="340" />
+        <mass value="${mass_base}" />
         <origin xyz="0 0 0" />
-        <inertia ixx="${mass_base/12.0 * (base_y_size*base_y_size + base_z_size*base_z_size)}" ixy="0" ixz="0"
-                 iyy="${mass_base/12.0 * (base_x_size*base_x_size + base_z_size*base_z_size)}" iyz="0"
-                 izz="${mass_base/12.0 * (base_y_size*base_y_size + base_x_size*base_x_size)}" />
+        <inertia ixx="0.21666666666666667" ixy="0" ixz="0"
+                 iyy="0.8416666666666667" iyz="0"
+                 izz="1.0416666666666667" />
       </inertial>
     </link>

File: robucar_description/urdf/wheel.xacro (robot description, xacro)
@@ -5,5 +5,5 @@
   <xacro:property name="wheel_length" value="0.1" />
   <xacro:property name="wheel_radius" value="0.28" />
-  <xacro:property name="mass_wheel" value="5.0" />
+  <xacro:property name="mass_wheel" value="0.1" />
   <xacro:macro name="wheel" params="wheel_prefix parent_link left_right *joint_origin">
     <gazebo reference="${wheel_prefix}_wheel_link">
@@ -13,11 +13,11 @@
 			<inertial>
         <mass value="${mass_wheel}" />
-        <origin xyz="0 0 0" rpy="${M_PI/2}  0 0" />
-        <!--<inertia ixx="1.0" ixy="0" ixz="0"
-                 iyy="1.0" iyz="0"
-                 izz="1.0"/>-->
-        <inertia  ixx="${mass_wheel/4.0*(wheel_radius*wheel_radius+wheel_length*wheel_length/3.0)}" ixy="0" ixz="0"
+        <origin xyz="0 0 0" rpy="${M_PI/2} 0 0" />
+        <inertia ixx="0.0030791666666666667" ixy="0" ixz="0"
+                 iyy="0.0030791666666666667" iyz="0"
+                 izz="0.005625"/>
+        <!--<inertia  ixx="${mass_wheel/4.0*(wheel_radius*wheel_radius+wheel_length*wheel_length/3.0)}" ixy="0" ixz="0"
                   iyy="${mass_wheel*wheel_radius*wheel_radius/2.0}" iyz="0"
-                  izz="${mass_wheel/4.0*(wheel_radius*wheel_radius+wheel_length*wheel_length/3.0)}" />
+                  izz="${mass_wheel/4.0*(wheel_radius*wheel_radius+wheel_length*wheel_length/3.0)}" />-->
       </inertial>
 			<visual>
@@ -33,10 +33,10 @@
 			<collision>
 				<origin xyz="0 0 0" rpy="${M_PI/2} 0 0" />
-				<geometry>
-					<cylinder length="${wheel_length}" radius="${wheel_radius}" />
+        <geometry>
+          <cylinder length="${wheel_length}" radius="${wheel_radius}" />
 				</geometry>
 			</collision>
 		</link>
-		<gazebo reference="${wheel_prefix}_wheel_link">
+    <!--<gazebo reference="${wheel_prefix}_wheel_link">
 			<mu1 value="1.0"/>
 			<mu2 value="1.0"/>
@@ -44,5 +44,5 @@
 			<kd value="1.0" />
 			<fdir1 value="1 0 0"/>
-		</gazebo>
+    </gazebo>-->
 		<joint name="${wheel_prefix}_wheel" type="continuous">
       <parent link="${parent_link}"/>

File: robucar_description/urdf/wheel_steered.xacro (robot description, xacro)
@@ -3,5 +3,5 @@
   <xacro:property name="steering_link_y" value="0.05" />
   <xacro:property name="steering_link_xz" value="0.1" />
-  <xacro:property name="steering_link_mass" value="30.0" />
+  <xacro:property name="steering_link_mass" value="0.4" />
   <xacro:include filename="$(find robucar_description)/urdf/wheel.xacro" />
   <xacro:macro name="wheel_steered" params="wheel_prefix parent_link wheel_origin_y left_right *joint_origin ">
@@ -19,19 +19,20 @@
         <mass value="${steering_link_mass}" />
         <origin xyz="0 0 0" />
-        <!--<inertia ixx="1.0" ixy="0" ixz="0"
-                 iyy="1.0" iyz="0"
-                 izz="1.0"/>-->
-        <inertia  ixx="${steering_link_mass/12.0 * (steering_link_y*steering_link_y + steering_link_xz*steering_link_xz)}" ixy="0" ixz="0"
+        <inertia ixx="0.0030791666666666667" ixy="0" ixz="0"
+                 iyy="0.0030791666666666667" iyz="0"
+                 izz="0.0030791666666666667"/>
+        <!--<inertia  ixx="${steering_link_mass/12.0 * (steering_link_y*steering_link_y + steering_link_xz*steering_link_xz)}" ixy="0" ixz="0"
                   iyy="${steering_link_mass/12.0 * (steering_link_xz*steering_link_xz + steering_link_xz*steering_link_xz)}" iyz="0"
-                  izz="${steering_link_mass/12.0 * (steering_link_y*steering_link_y + steering_link_xz*steering_link_xz)}" />
+                  izz="${steering_link_mass/12.0 * (steering_link_y*steering_link_y + steering_link_xz*steering_link_xz)}" />-->
       </inertial>
     </link>
     <joint name="${wheel_prefix}_steering_joint" type="revolute">
-      <limit lower="${-M_PI/6}" upper="${M_PI/6}" effort="1000.0" velocity="2.0"/>
+      <limit lower="${-M_PI/6}" upper="${M_PI/6}" effort="1000.0" velocity="1.0"/>
       <axis xyz="0 0 1"/>
       <parent link="${parent_link}"/>
       <child link="${wheel_prefix}_steering"/>
       <xacro:insert_block name="joint_origin"/>
-      <dynamics damping="0.7"/>
+      <!--<dynamics damping="0.7"/>-->
+      <dynamics damping="10.0" friction="20.0" />
     </joint>
     <transmission name="${wheel_prefix}_steering_trans" type="SimpleTransmission">

Commit message: Add true mass

File: robucar_description/urdf/chassis.xacro (robot description, xacro)
@@ -2,5 +2,5 @@
 <robot xmlns:xacro="http://www.ros.org/wiki/xacro" name="chassis">
   <!-- Base Properties -->
-  <xacro:property name="mass_base" value="10" />
+  <xacro:property name="mass_base" value="340" />
   <xacro:property name="base_x_size" value="1.66000" />
   <xacro:property name="base_y_size" value="0.60000" />
@@ -49,7 +49,10 @@
         <mass value="${mass_base}" />
         <origin xyz="0 0 0" />
-        <inertia ixx="0.21666666666666667" ixy="0" ixz="0"
+        <!--<inertia ixx="0.21666666666666667" ixy="0" ixz="0"
                  iyy="0.8416666666666667" iyz="0"
-                 izz="1.0416666666666667" />
+                 izz="1.0416666666666667" />-->
+        <inertia ixx="${mass_base/12.0 * (base_y_size*base_y_size + base_z_size*base_z_size)}" ixy="0" ixz="0"
+                        iyy="${mass_base/12.0 * (base_x_size*base_x_size + base_z_size*base_z_size)}" iyz="0"
+                        izz="${mass_base/12.0 * (base_y_size*base_y_size + base_x_size*base_x_size)}" />
       </inertial>
     </link>

File: robucar_description/urdf/wheel.xacro (robot description, xacro)
@@ -38,11 +38,11 @@
 			</collision>
 		</link>
-    <!--<gazebo reference="${wheel_prefix}_wheel_link">
-			<mu1 value="1.0"/>
-			<mu2 value="1.0"/>
-			<kp value="10000000.0" />
+    <gazebo reference="${wheel_prefix}_wheel_link">
+      <mu1 value="1.0"/>
+      <mu2 value="1.0"/>
+      <kp value="10000000.0" />
 			<kd value="1.0" />
-			<fdir1 value="1 0 0"/>
-    </gazebo>-->
+      <fdir1 value="1 0 0"/>
+    </gazebo>
 		<joint name="${wheel_prefix}_wheel" type="continuous">
       <parent link="${parent_link}"/>

Commit message: Revert "Add true mass"
This reverts commit 0715afc7c22f9218ee5e2233bc14d9fca45b3a7b.

File: robucar_description/urdf/chassis.xacro (robot description, xacro)
@@ -2,5 +2,5 @@
 <robot xmlns:xacro="http://www.ros.org/wiki/xacro" name="chassis">
   <!-- Base Properties -->
-  <xacro:property name="mass_base" value="340" />
+  <xacro:property name="mass_base" value="10" />
   <xacro:property name="base_x_size" value="1.66000" />
   <xacro:property name="base_y_size" value="0.60000" />
@@ -49,10 +49,7 @@
         <mass value="${mass_base}" />
         <origin xyz="0 0 0" />
-        <!--<inertia ixx="0.21666666666666667" ixy="0" ixz="0"
+        <inertia ixx="0.21666666666666667" ixy="0" ixz="0"
                  iyy="0.8416666666666667" iyz="0"
-                 izz="1.0416666666666667" />-->
-        <inertia ixx="${mass_base/12.0 * (base_y_size*base_y_size + base_z_size*base_z_size)}" ixy="0" ixz="0"
-                        iyy="${mass_base/12.0 * (base_x_size*base_x_size + base_z_size*base_z_size)}" iyz="0"
-                        izz="${mass_base/12.0 * (base_y_size*base_y_size + base_x_size*base_x_size)}" />
+                 izz="1.0416666666666667" />
       </inertial>
     </link>

File: robucar_description/urdf/wheel.xacro (robot description, xacro)
@@ -38,11 +38,11 @@
 			</collision>
 		</link>
-    <gazebo reference="${wheel_prefix}_wheel_link">
-      <mu1 value="1.0"/>
-      <mu2 value="1.0"/>
-      <kp value="10000000.0" />
+    <!--<gazebo reference="${wheel_prefix}_wheel_link">
+			<mu1 value="1.0"/>
+			<mu2 value="1.0"/>
+			<kp value="10000000.0" />
 			<kd value="1.0" />
-      <fdir1 value="1 0 0"/>
-    </gazebo>
+			<fdir1 value="1 0 0"/>
+    </gazebo>-->
 		<joint name="${wheel_prefix}_wheel" type="continuous">
       <parent link="${parent_link}"/>

Commit message: Working gps loc with robot_localization package in gazebo

File: robucar_description/urdf/chassis.xacro (robot description, xacro)
@@ -11,5 +11,5 @@
   <xacro:property name="ground_clearance" value="0.19" />
   <xacro:property name="wheel_x_offset" value="0.0" />
-  <xacro:property name="wheel_y_offset" value="0.0" />
+  <xacro:property name="wheel_y_offset" value="0.1" />
   <!-- LIDAR Properties -->
   <xacro:property name="lidar_ground_clearance" value="0.69" />

File: robucar_gazebo/urdf/robucar.gazebo.xacro (robot description, xacro)
@@ -27,5 +27,5 @@
           <referenceLatitude>45.76327</referenceLatitude>
           <referenceLongitude>3.1094</referenceLongitude>
-          <referenceHeading>0</referenceHeading>
+          <referenceHeading>90.0</referenceHeading>
           <referenceAltitude>400</referenceAltitude>
           <drift>0.05 0.05 0.05</drift>

Commit message: Add lidar frame link to use in simulation

File: robucar_description/urdf/chassis.xacro (robot description, xacro)
@@ -14,5 +14,5 @@
   <!-- LIDAR Properties -->
   <xacro:property name="lidar_ground_clearance" value="0.69" />
-  <xacro:property name="lidar_x_offset" value="0.4" />
+  <xacro:property name="lidar_x_offset" value="0.9" />
   <xacro:macro name="chassis">
     <!-- Base footprint is on the ground under the robot -->

File: robucar_description/urdf/robucar_4ws.urdf.xacro (robot description, xacro)
@@ -30,9 +30,10 @@
     </xacro:wheel_steered>
     <xacro:if value="$(arg laser_enabled)">
-      <!-- Hokuyo UTM-30LX mounted upside down below the body -->
-      <!--<xacro:include filename="$(find urg_description)/urdf/hokuyo_utm30lx.urdf.xacro" />
-      <xacro:hokuyo_utm30lx name="laser0" parent="base_link" ros_topic="scan" update_rate="40" ray_count="1081" min_angle="-135" max_angle="135">
-        <origin xyz="${lidar_x_offset} 0.0 ${lidar_ground_clearance - base_z_size/2 - ground_clearance}" rpy="0 0 0"/>
-      </xacro:hokuyo_utm30lx>-->
+      <link name="base_laser"/>
+      <joint name="laser_joint" type="fixed">
+        <origin xyz="${lidar_x_offset} 0.0 ${lidar_ground_clearance - base_z_size/2 - ground_clearance}" rpy="0 0 0" />
+        <parent link="base_link" />
+        <child link="base_laser" />
+      </joint>
     </xacro:if>
     <xacro:if value="$(arg camera_enabled)">
