Commit message: Update wheel steered for gazebo

File: robucar_description/urdf/wheel_steered.xacro (robot description, xacro)
@@ -3,8 +3,11 @@
   <xacro:include filename="$(find robucar_description)/urdf/wheel.xacro" />
   <xacro:macro name="wheel_steered" params="wheel_prefix parent_link *joint_origin">
-    <xacro:wheel wheel_prefix="${wheel_prefix}" parent_link="${wheel_prefix}_steering">
-      <origin xyz="0 0 0" rpy="0 0 0" />
-    </xacro:wheel>
-    <link name="${wheel_prefix}_steering"/>
+    <link name="${wheel_prefix}_steering">
+      <inertial>
+        <mass value="0.1" />
+        <origin xyz="0 0 0" />
+        <inertia  ixx="0.0" ixy="0" ixz="0" iyy="0.0" iyz="0" izz="0.0" />
+      </inertial>
+    </link>
     <joint name="${wheel_prefix}_steering_joint" type="revolute">
       <limit lower="-1.57075" upper="1.57075" effort="-1" velocity="-1"/>
@@ -14,4 +17,16 @@
       <xacro:insert_block name="joint_origin"/>
     </joint>
+    <transmission name="${wheel_prefix}_steering_trans" type="SimpleTransmission">
+      <type>transmission_interface/SimpleTransmission</type>
+      <actuator name="${wheel_prefix}_steering_motor">
+        <mechanicalReduction>1</mechanicalReduction>
+      </actuator>
+      <joint name="${wheel_prefix}_steering_joint">
+        <hardwareInterface>PositionJointInterface</hardwareInterface>
+      </joint>
+    </transmission>
+    <xacro:wheel wheel_prefix="${wheel_prefix}" parent_link="${wheel_prefix}_steering">
+      <origin xyz="0 0 0" rpy="0 0 0" />
+    </xacro:wheel>
   </xacro:macro>
 </robot>

Commit message: Remove damping on steering

File: robucar_description/urdf/wheel_steered.xacro (robot description, xacro)
@@ -33,5 +33,4 @@
       <child link="${wheel_prefix}_steering"/>
       <xacro:insert_block name="joint_origin"/>
-      <dynamics damping="0.7"/>
     </joint>
     <transmission name="${wheel_prefix}_steering_trans" type="SimpleTransmission">

Commit message: Clean scripts

File: robucar_description/urdf/wheel_steered.xacro (robot description, xacro)
@@ -33,4 +33,5 @@
       <child link="${wheel_prefix}_steering"/>
       <xacro:insert_block name="joint_origin"/>
+      <dynamics damping="0.7"/>
     </joint>
     <transmission name="${wheel_prefix}_steering_trans" type="SimpleTransmission">

Commit message: Fix steering oscillation on gazebo7 and enable twist for 4ws

File: robucar_description/urdf/wheel_steered.xacro (robot description, xacro)
@@ -3,5 +3,5 @@
   <xacro:property name="steering_link_y" value="0.05" />
   <xacro:property name="steering_link_xz" value="0.1" />
-  <xacro:property name="steering_link_mass" value="5.0" />
+  <xacro:property name="steering_link_mass" value="30.0" />
   <xacro:include filename="$(find robucar_description)/urdf/wheel.xacro" />
   <xacro:macro name="wheel_steered" params="wheel_prefix parent_link wheel_origin_y left_right *joint_origin ">

Commit message: remove damping

File: robucar_description/urdf/wheel_steered.xacro (robot description, xacro)
@@ -33,5 +33,4 @@
       <child link="${wheel_prefix}_steering"/>
       <xacro:insert_block name="joint_origin"/>
-      <dynamics damping="0.7"/>
       <!--<dynamics damping="10.0" friction="20.0" />-->
     </joint>
