Commit message: Add true value in robucar urdf (for robufast)

File: robucar_description/urdf/robucar.urdf.xacro (robot description, xacro)
@@ -7,15 +7,18 @@
   <xacro:property name="M_PI" value="3.14159"/>
   <!-- Base Size -->
-  <xacro:property name="base_x_size" value="0.50000" />
-  <xacro:property name="base_y_size" value="0.37000" />
-  <xacro:property name="base_z_size" value="0.17000" />
+  <xacro:property name="base_x_size" value="1.66000" />
+  <xacro:property name="base_y_size" value="0.60000" />
+  <xacro:property name="base_z_size" value="0.66000" />
   <!-- Wheel Mounting Positions -->
-  <xacro:property name="wheelbase" value="0.35" />
-  <xacro:property name="track" value="0.48" />
-  <xacro:property name="wheel_vertical_offset" value="-0.06" />
-  <xacro:property name="wheel_x_offset" value="-0.02" />
+  <xacro:property name="wheelbase" value="1.22" />
+  <xacro:property name="track" value="1.23" />
+  <xacro:property name="ground_clearance" value="0.19" />
+  <xacro:property name="wheel_x_offset" value="0.0" />
   <!-- Wheel Properties -->
-  <xacro:property name="wheel_length" value="0.09" />
-  <xacro:property name="wheel_radius" value="0.13" />
+  <xacro:property name="wheel_length" value="0.1" />
+  <xacro:property name="wheel_radius" value="0.28" />
+  <!-- LIDAR Properties -->
+  <xacro:property name="lidar_ground_clearance" value="0.69" />
+  <xacro:property name="lidar_x_offset" value="0.4" />
   <xacro:macro name="robucar">
     <!-- Base footprint is on the ground under the robot -->
@@ -41,5 +44,5 @@
     </link>
     <joint name="base_footprint_joint" type="fixed">
-      <origin xyz="0 0 ${-wheel_vertical_offset + wheel_radius}" rpy="0 0 0" />
+      <origin xyz="0 0 ${ground_clearance + base_z_size/2}" rpy="0 0 0" />
       <child link="base_link" />
       <parent link="base_footprint" />
@@ -48,7 +51,9 @@
     <link name="inertial_link">
       <inertial>
-        <mass value="33.455" />
+        <mass value="330" />
         <origin xyz="-0.08748 -0.00085 0.09947" />
-        <inertia ixx="0.6022" ixy="-0.02364" ixz="-0.1197" iyy="1.7386" iyz="-0.001544" izz="2.0296" />
+        <inertia ixx="0.6022" ixy="-0.02364" ixz="-0.1197"
+                 iyy="1.7386" iyz="-0.001544"
+                 izz="2.0296" />
       </inertial>
     </link>
@@ -67,4 +72,16 @@
     <!-- Wheel macros -->
     <xacro:wheel_steered wheel_prefix="front_left" parent_link="base_link">
+      <origin xyz="${wheelbase/2+wheel_x_offset} ${track/2} ${-base_z_size/2 + wheel_radius - ground_clearance}" rpy="0 0 0" />
+    </xacro:wheel_steered>
+    <xacro:wheel_steered wheel_prefix="front_right" parent_link="base_link">
+      <origin xyz="${wheelbase/2+wheel_x_offset} ${-track/2} ${-base_z_size/2 + wheel_radius - ground_clearance}" rpy="0 0 0" />
+    </xacro:wheel_steered>
+    <xacro:wheel wheel_prefix="rear_left" parent_link="base_link">
+      <origin xyz="${-wheelbase/2+wheel_x_offset} ${track/2} ${-base_z_size/2 + wheel_radius - ground_clearance}" rpy="0 0 0" />
+    </xacro:wheel>
+    <xacro:wheel wheel_prefix="rear_right" parent_link="base_link">
+      <origin xyz="${-wheelbase/2+wheel_x_offset} ${-track/2} ${-base_z_size/2 + wheel_radius - ground_clearance}" rpy="0 0 0" />
+    </xacro:wheel>
+    <!--<xacro:wheel_steered wheel_prefix="front_left" parent_link="base_link">
       <origin xyz="${wheelbase/2+wheel_x_offset} ${track/2} ${wheel_vertical_offset}" rpy="0 0 0" />
     </xacro:wheel_steered>
@@ -77,15 +94,11 @@
     <xacro:wheel_steered wheel_prefix="rear_right" parent_link="base_link">
       <origin xyz="${-wheelbase/2+wheel_x_offset} ${-track/2} ${wheel_vertical_offset}" rpy="0 0 0" />
-    </xacro:wheel_steered>
+    </xacro:wheel_steered>-->
     <xacro:if value="$(arg laser_enabled)">
       <!-- Hokuyo UTM-30LX mounted upside down below the body -->
       <!--<xacro:include filename="$(find urg_description)/urdf/hokuyo_utm30lx.urdf.xacro" />
       <xacro:hokuyo_utm30lx name="laser0" parent="base_link" ros_topic="scan" update_rate="40" ray_count="1081" min_angle="-135" max_angle="135">
-        <origin xyz="0.35 0.0 0.0" rpy="${M_PI} 0 0"/>
+        <origin xyz="${lidar_x_offset} 0.0 ${lidar_ground_clearance - base_z_size/2 - ground_clearance}" rpy="0 0 0"/>
       </xacro:hokuyo_utm30lx>-->
-      <!--<xacro:include filename="$(find urg_description)/urdf/hokuyo_urg_04lx_ug01_laser.urdf.xacro" />
-      <xacro:hokuyo_urg_04lx_ug01_laser name="laser0" parent="base_link" ros_topic="scan" update_rate="40" min_angle="-135" max_angle="135">
-        <origin xyz="0.35 0.0 0.0" rpy="${M_PI} 0 0"/>
-      </xacro:hokuyo_urg_04lx_ug01_laser>-->
     </xacro:if>
     <xacro:if value="$(arg camera_enabled)">

File: robucar_description/urdf/wheel.xacro (robot description, xacro)
@@ -10,7 +10,9 @@
 		<link name="${wheel_prefix}_wheel_link">
 			<inertial>
-				<mass value="2.637" />
+        <mass value="4.0" />
 				<origin xyz="0 0 0" />
-				<inertia  ixx="0.02467" ixy="0" ixz="0" iyy="0.02467" iyz="0" izz="0.04411" />
+        <inertia  ixx="1.0" ixy="0" ixz="0"
+                  iyy="1.0" iyz="0"
+                  izz="1.0" />
 			</inertial>
 			<visual>

File: robucar_description/urdf/wheel_steered.xacro (robot description, xacro)
@@ -7,9 +7,11 @@
         <mass value="0.1" />
         <origin xyz="0 0 0" />
-        <inertia  ixx="0.0" ixy="0" ixz="0" iyy="0.0" iyz="0" izz="0.0" />
+        <inertia  ixx="1.0" ixy="0" ixz="0"
+                  iyy="1.0" iyz="0"
+                  izz="1.0" />
       </inertial>
     </link>
     <joint name="${wheel_prefix}_steering_joint" type="revolute">
-      <limit lower="-1.57075" upper="1.57075" effort="-1" velocity="-1"/>
+      <limit lower="${-M_PI/4}" upper="${M_PI/4}" effort="-1" velocity="-1"/>
       <axis xyz="0 0 1"/>
       <parent link="${parent_link}"/>
@@ -20,4 +22,5 @@
       <type>transmission_interface/SimpleTransmission</type>
       <actuator name="${wheel_prefix}_steering_motor">
+        <hardwareInterface>PositionJointInterface</hardwareInterface>
         <mechanicalReduction>1</mechanicalReduction>
       </actuator>

Commit message: Fix revolute joint with positive effort and velocity.
Change inertia moment and mass.

File: robucar_description/urdf/robucar.urdf.xacro (robot description, xacro)
@@ -6,5 +6,6 @@
   <xacro:include filename="$(find robucar_description)/urdf/wheel_steered.xacro" />
   <xacro:property name="M_PI" value="3.14159"/>
-  <!-- Base Size -->
+  <!-- Base Properties -->
+  <xacro:property name="mass_base" value="340" />
   <xacro:property name="base_x_size" value="1.66000" />
   <xacro:property name="base_y_size" value="0.60000" />
@@ -15,4 +16,5 @@
   <xacro:property name="ground_clearance" value="0.19" />
   <xacro:property name="wheel_x_offset" value="0.0" />
+  <xacro:property name="wheel_y_offset" value="0.05" />
   <!-- Wheel Properties -->
   <xacro:property name="wheel_length" value="0.1" />
@@ -51,9 +53,9 @@
     <link name="inertial_link">
       <inertial>
-        <mass value="330" />
-        <origin xyz="-0.08748 -0.00085 0.09947" />
-        <inertia ixx="0.6022" ixy="-0.02364" ixz="-0.1197"
-                 iyy="1.7386" iyz="-0.001544"
-                 izz="2.0296" />
+        <mass value="340" />
+        <origin xyz="0 0 0" />
+        <inertia ixx="${mass_base/12.0 * (base_y_size*base_y_size + base_z_size*base_z_size)}" ixy="0" ixz="0"
+                 iyy="${mass_base/12.0 * (base_x_size*base_x_size + base_z_size*base_z_size)}" iyz="0"
+                 izz="${mass_base/12.0 * (base_y_size*base_y_size + base_x_size*base_x_size)}" />
       </inertial>
     </link>
@@ -71,9 +73,9 @@
     </joint>
     <!-- Wheel macros -->
-    <xacro:wheel_steered wheel_prefix="front_left" parent_link="base_link">
-      <origin xyz="${wheelbase/2+wheel_x_offset} ${track/2} ${-base_z_size/2 + wheel_radius - ground_clearance}" rpy="0 0 0" />
+    <xacro:wheel_steered wheel_prefix="front_left" parent_link="base_link" wheel_origin_y="${wheel_y_offset}">
+      <origin xyz="${wheelbase/2+wheel_x_offset} ${track/2-wheel_y_offset} ${-base_z_size/2 + wheel_radius - ground_clearance}" rpy="0 0 0" />
     </xacro:wheel_steered>
-    <xacro:wheel_steered wheel_prefix="front_right" parent_link="base_link">
-      <origin xyz="${wheelbase/2+wheel_x_offset} ${-track/2} ${-base_z_size/2 + wheel_radius - ground_clearance}" rpy="0 0 0" />
+    <xacro:wheel_steered wheel_prefix="front_right" parent_link="base_link" wheel_origin_y="${-wheel_y_offset}">
+      <origin xyz="${wheelbase/2+wheel_x_offset} ${-track/2+wheel_y_offset} ${-base_z_size/2 + wheel_radius - ground_clearance}" rpy="0 0 0" />
     </xacro:wheel_steered>
     <xacro:wheel wheel_prefix="rear_left" parent_link="base_link">

File: robucar_description/urdf/wheel.xacro (robot description, xacro)
@@ -4,4 +4,5 @@
   <xacro:property name="wheel_length" default="0.09" />
   <xacro:property name="wheel_radius" default="0.13" />-->
+  <xacro:property name="mass_wheel" value="5.0" />
   <xacro:macro name="wheel" params="wheel_prefix parent_link *joint_origin">
     <gazebo reference="${wheel_prefix}_wheel_link">
@@ -10,10 +11,13 @@
 		<link name="${wheel_prefix}_wheel_link">
 			<inertial>
-        <mass value="4.0" />
-				<origin xyz="0 0 0" />
-        <inertia  ixx="1.0" ixy="0" ixz="0"
-                  iyy="1.0" iyz="0"
-                  izz="1.0" />
-			</inertial>
+        <mass value="${mass_wheel}" />
+        <origin xyz="0 0 0" rpy="${M_PI/2}  0 0" />
+        <!--<inertia ixx="1.0" ixy="0" ixz="0"
+                 iyy="1.0" iyz="0"
+                 izz="1.0"/>-->
+        <inertia  ixx="${mass_wheel/4.0*(wheel_radius*wheel_radius+wheel_length*wheel_length/3.0)}" ixy="0" ixz="0"
+                  iyy="${mass_wheel*wheel_radius*wheel_radius/2.0}" iyz="0"
+                  izz="${mass_wheel/4.0*(wheel_radius*wheel_radius+wheel_length*wheel_length/3.0)}" />
+      </inertial>
 			<visual>
 				<origin xyz="0 0 0" rpy="${M_PI/2}  0 0" />

File: robucar_description/urdf/wheel_steered.xacro (robot description, xacro)
@@ -1,21 +1,37 @@
 <?xml version="1.0"?>
 <robot xmlns:xacro="http://ros.org/wiki/xacro" name="wheel_steered">
+  <xacro:property name="steering_link_y" value="0.05" />
+  <xacro:property name="steering_link_xz" value="0.1" />
+  <xacro:property name="steering_link_mass" value="5.0" />
   <xacro:include filename="$(find robucar_description)/urdf/wheel.xacro" />
-  <xacro:macro name="wheel_steered" params="wheel_prefix parent_link *joint_origin">
+  <xacro:macro name="wheel_steered" params="wheel_prefix parent_link wheel_origin_y *joint_origin ">
     <link name="${wheel_prefix}_steering">
+      <visual>
+        <origin xyz="0 ${-wheel_origin_y} 0" rpy="0 0 0"/>
+        <geometry>
+          <box size="0.05 ${steering_link_y} 0.05"/>
+        </geometry>
+        <material name="blue">
+          <color rgba="0.2 0.2 0.6 1"/>
+        </material>
+      </visual>
       <inertial>
-        <mass value="0.1" />
-        <origin xyz="0 0 0" />
-        <inertia  ixx="1.0" ixy="0" ixz="0"
-                  iyy="1.0" iyz="0"
-                  izz="1.0" />
+        <mass value="${steering_link_mass}" />
+        <origin xyz="0 ${-wheel_origin_y} 0" />
+        <!--<inertia ixx="1.0" ixy="0" ixz="0"
+                 iyy="1.0" iyz="0"
+                 izz="1.0"/>-->
+        <inertia  ixx="${steering_link_mass/12.0 * (steering_link_y*steering_link_y + steering_link_xz*steering_link_xz)}" ixy="0" ixz="0"
+                  iyy="${steering_link_mass/12.0 * (steering_link_xz*steering_link_xz + steering_link_xz*steering_link_xz)}" iyz="0"
+                  izz="${steering_link_mass/12.0 * (steering_link_y*steering_link_y + steering_link_xz*steering_link_xz)}" />
       </inertial>
     </link>
     <joint name="${wheel_prefix}_steering_joint" type="revolute">
-      <limit lower="${-M_PI/4}" upper="${M_PI/4}" effort="-1" velocity="-1"/>
+      <limit lower="${-M_PI/6}" upper="${M_PI/6}" effort="1000.0" velocity="2.0"/>
       <axis xyz="0 0 1"/>
       <parent link="${parent_link}"/>
       <child link="${wheel_prefix}_steering"/>
       <xacro:insert_block name="joint_origin"/>
+      <dynamics damping="0.7"/>
     </joint>
     <transmission name="${wheel_prefix}_steering_trans" type="SimpleTransmission">
@@ -30,5 +46,5 @@
     </transmission>
     <xacro:wheel wheel_prefix="${wheel_prefix}" parent_link="${wheel_prefix}_steering">
-      <origin xyz="0 0 0" rpy="0 0 0" />
+      <origin xyz="0 ${wheel_origin_y} 0" rpy="0 0 0" />
     </xacro:wheel>
   </xacro:macro>

Commit message: Add robucar bringup and velodyne in simulation

File: robucar_description/urdf/robucar.urdf.xacro (robot description, xacro)
@@ -120,4 +120,10 @@
       </joint>
     </xacro:if>
+    <!--<link name="velodyne"/>
+    <joint name="velodyne_joint" type="fixed">
+      <origin xyz="0.0 0.0 1.0" rpy="0 0 0" />
+      <parent link="base_link" />
+      <child link="velodyne" />
+    </joint>-->
   </xacro:macro>
 </robot>

File: robucar_gazebo/urdf/robucar.gazebo.xacro (robot description, xacro)
@@ -76,4 +76,35 @@
       </sensor>
     </gazebo>-->
+    <!--<gazebo reference="velodyne">
+        <sensor type="ray" name="velodyne_sensor">
+          <pose>0.0 0.0 0.0 0.0 0 0</pose>
+          <visualize>false</visualize>
+          <update_rate>5</update_rate>
+          <ray>
+            <scan>
+              <horizontal>
+                <samples>720</samples>
+                <min_angle>-3.13</min_angle>
+                <max_angle>3.14</max_angle>
+              </horizontal>
+              <vertical>
+                <samples>16</samples>
+                <min_angle>-0.13</min_angle>
+                <max_angle>0.13</max_angle>
+              </vertical>
+            </scan>
+            <range>
+              <min>0.30</min>
+              <max>30.0</max>
+            </range>
+          </ray>
+          <plugin name="gazebo_ros_head_hokuyo_controller" filename="libgazebo_ros_block_laser.so">
+            <topicName>scan_velodyne</topicName>
+            <updateRate>5</updateRate>
+            <frameName>/velodyne</frameName>
+            <alwaysOn>true</alwaysOn>
+          </plugin>
+        </sensor>
+    </gazebo>-->
   </xacro:macro>
 </robot>

Commit message: Load robufast meshes in urdf

File: robucar_description/urdf/robucar.urdf.xacro (robot description, xacro)
@@ -32,6 +32,8 @@
     <link name="base_link">
       <visual>
+        <origin xyz="-0.5 -0.04 -0.06" rpy="0 0 ${M_PI/2.0}" />
         <geometry>
-          <box size="${base_x_size} ${base_y_size} ${base_z_size}"/>
+          <!--<box size="${base_x_size} ${base_y_size} ${base_z_size}"/>-->
+          <mesh filename="package://robucar_description/meshes/robufast_frame_0_72.dae"/>
         </geometry>
         <material name="grey">
@@ -73,14 +75,14 @@
     </joint>
     <!-- Wheel macros -->
-    <xacro:wheel_steered wheel_prefix="front_left" parent_link="base_link" wheel_origin_y="${wheel_y_offset}">
+    <xacro:wheel_steered wheel_prefix="front_left" parent_link="base_link" wheel_origin_y="${wheel_y_offset}" left_right="-1">
       <origin xyz="${wheelbase/2+wheel_x_offset} ${track/2-wheel_y_offset} ${-base_z_size/2 + wheel_radius - ground_clearance}" rpy="0 0 0" />
     </xacro:wheel_steered>
-    <xacro:wheel_steered wheel_prefix="front_right" parent_link="base_link" wheel_origin_y="${-wheel_y_offset}">
+    <xacro:wheel_steered wheel_prefix="front_right" parent_link="base_link" wheel_origin_y="${-wheel_y_offset}" left_right="1">
       <origin xyz="${wheelbase/2+wheel_x_offset} ${-track/2+wheel_y_offset} ${-base_z_size/2 + wheel_radius - ground_clearance}" rpy="0 0 0" />
     </xacro:wheel_steered>
-    <xacro:wheel wheel_prefix="rear_left" parent_link="base_link">
+    <xacro:wheel wheel_prefix="rear_left" parent_link="base_link" left_right="-1">
       <origin xyz="${-wheelbase/2+wheel_x_offset} ${track/2} ${-base_z_size/2 + wheel_radius - ground_clearance}" rpy="0 0 0" />
     </xacro:wheel>
-    <xacro:wheel wheel_prefix="rear_right" parent_link="base_link">
+    <xacro:wheel wheel_prefix="rear_right" parent_link="base_link" left_right="1">
       <origin xyz="${-wheelbase/2+wheel_x_offset} ${-track/2} ${-base_z_size/2 + wheel_radius - ground_clearance}" rpy="0 0 0" />
     </xacro:wheel>

File: robucar_description/urdf/wheel.xacro (robot description, xacro)
@@ -5,5 +5,5 @@
   <xacro:property name="wheel_radius" default="0.13" />-->
   <xacro:property name="mass_wheel" value="5.0" />
-  <xacro:macro name="wheel" params="wheel_prefix parent_link *joint_origin">
+  <xacro:macro name="wheel" params="wheel_prefix parent_link left_right *joint_origin">
     <gazebo reference="${wheel_prefix}_wheel_link">
       <material>Gazebo/Black</material>
@@ -21,7 +21,8 @@
       </inertial>
 			<visual>
-				<origin xyz="0 0 0" rpy="${M_PI/2}  0 0" />
+        <origin xyz="0 0 0" rpy="${left_right * M_PI/2}  0 0" />
 				<geometry>
-          <cylinder length="${wheel_length}" radius="${wheel_radius}"/>
+          <!--<cylinder length="${wheel_length}" radius="${wheel_radius}"/>-->
+          <mesh filename="package://robucar_description/meshes/robufast_wheel_d0_56.dae"/>
 				</geometry>
         <material name="black">

File: robucar_description/urdf/wheel_steered.xacro (robot description, xacro)
@@ -5,5 +5,5 @@
   <xacro:property name="steering_link_mass" value="5.0" />
   <xacro:include filename="$(find robucar_description)/urdf/wheel.xacro" />
-  <xacro:macro name="wheel_steered" params="wheel_prefix parent_link wheel_origin_y *joint_origin ">
+  <xacro:macro name="wheel_steered" params="wheel_prefix parent_link wheel_origin_y left_right *joint_origin ">
     <link name="${wheel_prefix}_steering">
       <visual>
@@ -45,5 +45,5 @@
       </joint>
     </transmission>
-    <xacro:wheel wheel_prefix="${wheel_prefix}" parent_link="${wheel_prefix}_steering">
+    <xacro:wheel wheel_prefix="${wheel_prefix}" parent_link="${wheel_prefix}_steering" left_right="${left_right}">
       <origin xyz="0 ${wheel_origin_y} 0" rpy="0 0 0" />
     </xacro:wheel>
