Commit message: [robucar_description] add common chassis file

File: robucar_description/urdf/robucar.urdf.xacro (robot description, xacro)
@@ -5,66 +5,15 @@
   <xacro:arg name="navsat_enabled" default="false" />
   <xacro:include filename="$(find robucar_description)/urdf/wheel_steered.xacro" />
+  <xacro:include filename="$(find robucar_description)/urdf/chassis.xacro" />
   <xacro:property name="M_PI" value="3.14159"/>
-  <!-- Base Properties -->
-  <xacro:property name="mass_base" value="340" />
-  <xacro:property name="base_x_size" value="1.66000" />
-  <xacro:property name="base_y_size" value="0.60000" />
-  <xacro:property name="base_z_size" value="0.66000" />
   <!-- Wheel Mounting Positions -->
-  <xacro:property name="wheelbase" value="1.22" />
-  <xacro:property name="track" value="1.23" />
   <xacro:property name="ground_clearance" value="0.19" />
   <xacro:property name="wheel_x_offset" value="0.0" />
   <xacro:property name="wheel_y_offset" value="0.05" />
-  <!-- Wheel Properties -->
-  <xacro:property name="wheel_length" value="0.1" />
-  <xacro:property name="wheel_radius" value="0.28" />
   <!-- LIDAR Properties -->
   <xacro:property name="lidar_ground_clearance" value="0.69" />
   <xacro:property name="lidar_x_offset" value="0.4" />
   <xacro:macro name="robucar">
-    <!-- Base footprint is on the ground under the robot -->
-    <link name="base_footprint"/>
-    <gazebo reference="base_link">
-      <material>Gazebo/Grey</material>
-    </gazebo>
-    <!-- Base link is the center of the robot's bottom plate -->
-    <link name="base_link">
-      <visual>
-        <origin xyz="-0.5 -0.04 -0.06" rpy="0 0 ${M_PI/2.0}" />
-        <geometry>
-          <!--<box size="${base_x_size} ${base_y_size} ${base_z_size}"/>-->
-          <mesh filename="package://robucar_description/meshes/robufast_frame_0_72.dae"/>
-        </geometry>
-        <material name="grey">
-          <color rgba="0.6 0.6 0.6 1"/>
-        </material>
-      </visual>
-      <collision>
-        <geometry>
-          <box size="${base_x_size} ${base_y_size} ${base_z_size}"/>
-        </geometry>
-      </collision>
-    </link>
-    <joint name="base_footprint_joint" type="fixed">
-      <origin xyz="0 0 ${ground_clearance + base_z_size/2}" rpy="0 0 0" />
-      <child link="base_link" />
-      <parent link="base_footprint" />
-    </joint>
-    <!-- Interial link stores the robot's inertial information -->
-    <link name="inertial_link">
-      <inertial>
-        <mass value="340" />
-        <origin xyz="0 0 0" />
-        <inertia ixx="${mass_base/12.0 * (base_y_size*base_y_size + base_z_size*base_z_size)}" ixy="0" ixz="0"
-                 iyy="${mass_base/12.0 * (base_x_size*base_x_size + base_z_size*base_z_size)}" iyz="0"
-                 izz="${mass_base/12.0 * (base_y_size*base_y_size + base_x_size*base_x_size)}" />
-      </inertial>
-    </link>
-    <joint name="inertial_joint" type="fixed">
-      <origin xyz="0 0 0" rpy="0 0 0" />
-      <parent link="base_link" />
-      <child link="inertial_link" />
-    </joint>
+    <xacro:chassis/>
     <!-- IMU Link is the standard mounting position for the IMU.-->
     <link name="imu_link"/>
@@ -87,16 +36,4 @@
       <origin xyz="${-wheelbase/2+wheel_x_offset} ${-track/2} ${-base_z_size/2 + wheel_radius - ground_clearance}" rpy="0 0 0" />
     </xacro:wheel>
-    <!--<xacro:wheel_steered wheel_prefix="front_left" parent_link="base_link">
-      <origin xyz="${wheelbase/2+wheel_x_offset} ${track/2} ${wheel_vertical_offset}" rpy="0 0 0" />
-    </xacro:wheel_steered>
-    <xacro:wheel_steered wheel_prefix="front_right" parent_link="base_link">
-      <origin xyz="${wheelbase/2+wheel_x_offset} ${-track/2} ${wheel_vertical_offset}" rpy="0 0 0" />
-    </xacro:wheel_steered>
-    <xacro:wheel_steered wheel_prefix="rear_left" parent_link="base_link">
-      <origin xyz="${-wheelbase/2+wheel_x_offset} ${track/2} ${wheel_vertical_offset}" rpy="0 0 0" />
-    </xacro:wheel_steered>
-    <xacro:wheel_steered wheel_prefix="rear_right" parent_link="base_link">
-      <origin xyz="${-wheelbase/2+wheel_x_offset} ${-track/2} ${wheel_vertical_offset}" rpy="0 0 0" />
-    </xacro:wheel_steered>-->
     <xacro:if value="$(arg laser_enabled)">
       <!-- Hokuyo UTM-30LX mounted upside down below the body -->

File: robucar_description/urdf/robucar_4ws.urdf.xacro (robot description, xacro)
@@ -5,64 +5,15 @@
   <xacro:arg name="navsat_enabled" default="false" />
   <xacro:include filename="$(find robucar_description)/urdf/wheel_steered.xacro" />
+  <xacro:include filename="$(find robucar_description)/urdf/chassis.xacro" />
   <xacro:property name="M_PI" value="3.14159"/>
-  <!-- Base Properties -->
-  <xacro:property name="mass_base" value="340" />
-  <xacro:property name="base_x_size" value="1.66000" />
-  <xacro:property name="base_y_size" value="0.60000" />
-  <xacro:property name="base_z_size" value="0.66000" />
   <!-- Wheel Mounting Positions -->
-  <xacro:property name="wheelbase" value="1.22" />
-  <xacro:property name="track" value="1.23" />
   <xacro:property name="ground_clearance" value="0.19" />
   <xacro:property name="wheel_x_offset" value="0.0" />
   <xacro:property name="wheel_y_offset" value="0.05" />
-  <!-- Wheel Properties -->
-  <xacro:property name="wheel_length" value="0.1" />
-  <xacro:property name="wheel_radius" value="0.28" />
   <!-- LIDAR Properties -->
   <xacro:property name="lidar_ground_clearance" value="0.69" />
   <xacro:property name="lidar_x_offset" value="0.4" />
   <xacro:macro name="robucar">
-    <!-- Base footprint is on the ground under the robot -->
-    <link name="base_footprint"/>
-    <gazebo reference="base_link">
-      <material>Gazebo/Grey</material>
-    </gazebo>
-    <!-- Base link is the center of the robot's bottom plate -->
-    <link name="base_link">
-      <visual>
-        <geometry>
-          <box size="${base_x_size} ${base_y_size} ${base_z_size}"/>
-        </geometry>
-        <material name="grey">
-          <color rgba="0.6 0.6 0.6 1"/>
-        </material>
-      </visual>
-      <collision>
-        <geometry>
-          <box size="${base_x_size} ${base_y_size} ${base_z_size}"/>
-        </geometry>
-      </collision>
-    </link>
-    <joint name="base_footprint_joint" type="fixed">
-      <origin xyz="0 0 ${ground_clearance + base_z_size/2}" rpy="0 0 0" />
-      <child link="base_link" />
-      <parent link="base_footprint" />
-    </joint>
-    <!-- Interial link stores the robot's inertial information -->
-    <link name="inertial_link">
-      <inertial>
-        <mass value="340" />
-        <origin xyz="0 0 0" />
-        <inertia ixx="${mass_base/12.0 * (base_y_size*base_y_size + base_z_size*base_z_size)}" ixy="0" ixz="0"
-                 iyy="${mass_base/12.0 * (base_x_size*base_x_size + base_z_size*base_z_size)}" iyz="0"
-                 izz="${mass_base/12.0 * (base_y_size*base_y_size + base_x_size*base_x_size)}" />
-      </inertial>
-    </link>
-    <joint name="inertial_joint" type="fixed">
-      <origin xyz="0 0 0" rpy="0 0 0" />
-      <parent link="base_link" />
-      <child link="inertial_link" />
-    </joint>
+    <xacro:chassis/>
     <!-- IMU Link is the standard mounting position for the IMU.-->
     <link name="imu_link"/>
@@ -73,14 +24,14 @@
     </joint>
     <!-- Wheel macros -->
-    <xacro:wheel_steered wheel_prefix="front_left" parent_link="base_link" wheel_origin_y="${wheel_y_offset}">
+    <xacro:wheel_steered wheel_prefix="front_left" parent_link="base_link" wheel_origin_y="${wheel_y_offset}"  left_right="-1">
       <origin xyz="${wheelbase/2+wheel_x_offset} ${track/2-wheel_y_offset} ${-base_z_size/2 + wheel_radius - ground_clearance}" rpy="0 0 0" />
     </xacro:wheel_steered>
-    <xacro:wheel_steered wheel_prefix="front_right" parent_link="base_link" wheel_origin_y="${-wheel_y_offset}">
+    <xacro:wheel_steered wheel_prefix="front_right" parent_link="base_link" wheel_origin_y="${-wheel_y_offset}"  left_right="1">
       <origin xyz="${wheelbase/2+wheel_x_offset} ${-track/2+wheel_y_offset} ${-base_z_size/2 + wheel_radius - ground_clearance}" rpy="0 0 0" />
     </xacro:wheel_steered>
-    <xacro:wheel_steered wheel_prefix="rear_left" parent_link="base_link" wheel_origin_y="${wheel_y_offset}">
+    <xacro:wheel_steered wheel_prefix="rear_left" parent_link="base_link" wheel_origin_y="${wheel_y_offset}"  left_right="-1">
       <origin xyz="${-wheelbase/2+wheel_x_offset} ${track/2-wheel_y_offset} ${-base_z_size/2 + wheel_radius - ground_clearance}" rpy="0 0 0" />
     </xacro:wheel_steered>
-    <xacro:wheel_steered wheel_prefix="rear_right" parent_link="base_link" wheel_origin_y="${-wheel_y_offset}">
+    <xacro:wheel_steered wheel_prefix="rear_right" parent_link="base_link" wheel_origin_y="${-wheel_y_offset}"  left_right="1">
       <origin xyz="${-wheelbase/2+wheel_x_offset} ${-track/2+wheel_y_offset} ${-base_z_size/2 + wheel_radius - ground_clearance}" rpy="0 0 0" />
     </xacro:wheel_steered>

File: robucar_description/urdf/wheel.xacro (robot description, xacro)
@@ -1,7 +1,8 @@
 <?xml version="1.0"?>
 <robot xmlns:xacro="http://www.ros.org/wiki/xacro" name="wheel">
-  <!--<xacro:property name="M_PI" default="3.14159"/>
-  <xacro:property name="wheel_length" default="0.09" />
-  <xacro:property name="wheel_radius" default="0.13" />-->
+  <!--<xacro:property name="M_PI" default="3.14159"/>-->
+  <!-- Wheel Properties -->
+  <xacro:property name="wheel_length" value="0.1" />
+  <xacro:property name="wheel_radius" value="0.28" />
   <xacro:property name="mass_wheel" value="5.0" />
   <xacro:macro name="wheel" params="wheel_prefix parent_link left_right *joint_origin">

Commit message: Change for use with mapping gazebo

File: robucar_description/urdf/robucar.urdf.xacro (robot description, xacro)
@@ -124,5 +124,5 @@
     <xacro:include filename="$(find velodyne_description)/urdf/HDL-32E.urdf.xacro"/>
     <HDL-32E parent="base_link" name="velodyne2" topic="/velodyne_points2">
-      <origin xyz="0 0 0.6" rpy="0 0 0" />
+      <origin xyz="${base_x_size/2-0.01} 0 ${base_z_size/2}" rpy="0 0 0" />
     </HDL-32E>
     </xacro:if>

File: robucar_gazebo/urdf/description.gazebo.xacro (robot description, xacro)
@@ -3,5 +3,5 @@
   <xacro:arg name="laser_enabled" default="false" />
   <xacro:arg name="camera_enabled" default="false" />
-  <xacro:arg name="navsat_enabled" default="false" />
+  <xacro:arg name="navsat_enabled" default="true" />
   <xacro:arg name="velodyne_enabled" default="false" />
   <xacro:include filename="$(find robucar_description)/urdf/robucar.urdf.xacro" />

File: robucar_gazebo/urdf/robucar.gazebo.xacro (robot description, xacro)
@@ -77,3 +77,37 @@
     </gazebo>-->
   </xacro:macro>
+<!--<xacro:if value="$(arg velodyne_enabled)">
+<gazebo reference="velodyne_link">
+    <sensor type="ray" name="velodyne_sensor">
+      <pose>0.0 0.0 0.0 0.0 0 0</pose>
+      <visualize>false</visualize>
+      <update_rate>10</update_rate>
+      <ray>
+        <scan>
+          <horizontal>
+            <samples>720</samples>
+            <min_angle>-3.13</min_angle>
+            <max_angle>3.14</max_angle>
+          </horizontal>
+          <vertical>
+            <samples>32</samples>
+            <min_angle>-0.53529248</min_angle>
+            <max_angle>0.18622663</max_angle>
+          </vertical>
+        </scan>
+        <range>
+          <min>0.05</min>
+          <max>70.0</max>
+          <resolution>0.02</resolution>
+        </range>
+      </ray>
+      <plugin name="gazebo_ros_head_hokuyo_controller" filename="libgazebo_ros_block_laser.so">
+        <topicName>scan_velodyne</topicName>
+        <updateRate>10</updateRate>
+        <frameName>/velodyne_link</frameName>
+        <alwaysOn>true</alwaysOn>
+      </plugin>
+    </sensor>
+    </gazebo>
+  </xacro:if>-->
 </robot>

Commit message: Allignement de urdf

File: robucar_description/urdf/robucar.urdf.xacro (robot description, xacro)
@@ -122,8 +122,8 @@
     </xacro:if>
     <xacro:if value="$(arg velodyne_enabled)">
-    <xacro:include filename="$(find velodyne_description)/urdf/HDL-32E.urdf.xacro"/>
-    <HDL-32E parent="base_link" name="velodyne2" topic="/velodyne_points2">
-      <origin xyz="${base_x_size/2-0.01} 0 ${base_z_size/2}" rpy="0 0 0" />
-    </HDL-32E>
+      <xacro:include filename="$(find velodyne_description)/urdf/HDL-32E.urdf.xacro"/>
+      <HDL-32E parent="base_link" name="velodyne2" topic="/velodyne_points2">
+        <origin xyz="${base_x_size/2-0.01} 0 ${base_z_size/2}" rpy="0 0 0" />
+      </HDL-32E>
     </xacro:if>
   </xacro:macro>

File: robucar_gazebo/urdf/robucar.gazebo.xacro (robot description, xacro)
@@ -77,37 +77,37 @@
     </gazebo>-->
   </xacro:macro>
-<!--<xacro:if value="$(arg velodyne_enabled)">
-<gazebo reference="velodyne_link">
-    <sensor type="ray" name="velodyne_sensor">
-      <pose>0.0 0.0 0.0 0.0 0 0</pose>
-      <visualize>false</visualize>
-      <update_rate>10</update_rate>
-      <ray>
-        <scan>
-          <horizontal>
-            <samples>720</samples>
-            <min_angle>-3.13</min_angle>
-            <max_angle>3.14</max_angle>
-          </horizontal>
-          <vertical>
-            <samples>32</samples>
-            <min_angle>-0.53529248</min_angle>
-            <max_angle>0.18622663</max_angle>
-          </vertical>
-        </scan>
-        <range>
-          <min>0.05</min>
-          <max>70.0</max>
-          <resolution>0.02</resolution>
-        </range>
-      </ray>
-      <plugin name="gazebo_ros_head_hokuyo_controller" filename="libgazebo_ros_block_laser.so">
-        <topicName>scan_velodyne</topicName>
-        <updateRate>10</updateRate>
-        <frameName>/velodyne_link</frameName>
-        <alwaysOn>true</alwaysOn>
-      </plugin>
-    </sensor>
-    </gazebo>
-  </xacro:if>-->
+<!--<xacro:if value="$(arg velodyne_enabled)">-->
+  <!--<gazebo reference="velodyne_link">
+      <sensor type="ray" name="velodyne_sensor">
+        <pose>0.0 0.0 0.0 0.0 0 0</pose>
+        <visualize>false</visualize>
+        <update_rate>10</update_rate>
+        <ray>
+          <scan>
+            <horizontal>
+              <samples>720</samples>
+              <min_angle>-3.13</min_angle>
+              <max_angle>3.14</max_angle>
+            </horizontal>
+            <vertical>
+              <samples>32</samples>
+              <min_angle>-0.53529248</min_angle>
+              <max_angle>0.18622663</max_angle>
+            </vertical>
+          </scan>
+          <range>
+            <min>0.05</min>
+            <max>70.0</max>
+            <resolution>0.02</resolution>
+          </range>
+        </ray>
+        <plugin name="gazebo_ros_head_hokuyo_controller" filename="libgazebo_ros_block_laser.so">
+          <topicName>velodyne_points2</topicName>
+          <updateRate>10</updateRate>
+          <frameName>/velodyne_link</frameName>
+          <alwaysOn>true</alwaysOn>
+        </plugin>
+      </sensor>
+  </gazebo>-->
+<!--</xacro:if>-->
 </robot>

Commit message: Update robucar simu config

File: robucar_description/urdf/robucar.urdf.xacro (robot description, xacro)
@@ -31,9 +31,11 @@
     </xacro:wheel>
     <xacro:if value="$(arg laser_enabled)">
-      <!-- Hokuyo UTM-30LX mounted upside down below the body -->
-      <!--<xacro:include filename="$(find urg_description)/urdf/hokuyo_utm30lx.urdf.xacro" />
-      <xacro:hokuyo_utm30lx name="laser0" parent="base_link" ros_topic="scan" update_rate="40" ray_count="1081" min_angle="-135" max_angle="135">
-        <origin xyz="${lidar_x_offset} 0.0 ${lidar_ground_clearance - base_z_size/2 - ground_clearance}" rpy="0 0 0"/>
-      </xacro:hokuyo_utm30lx>-->
+      <xacro:include filename="$(find lms1xx)/urdf/sick_lms1xx.urdf.xacro"/>
+      <xacro:sick_lms1xx />
+      <joint name="laser_joint" type="fixed">
+        <origin xyz="${lidar_x_offset} 0.0 ${lidar_ground_clearance - base_z_size/2 - ground_clearance}" rpy="0 0 0" />
+        <parent link="base_link" />
+        <child link="laser" />
+      </joint>
     </xacro:if>
     <xacro:if value="$(arg camera_enabled)">
@@ -46,10 +48,22 @@
     </xacro:if>
     <xacro:if value="$(arg navsat_enabled)">
-      <link name="navsat_link"/>
-      <joint name="navsat_joint" type="fixed">
-        <origin xyz="0.3 0 0.3" rpy="0 0 0" />
+      <link name="navsat_link">
+        <inertial>
+          <inertia ixx="0.00001" ixy="0.0" ixz="0.0" iyy="0.00001" iyz="0.0" izz="0.00001" />
+          <mass value="0.015" />  <!-- [kg] -->
+          <origin xyz="0 0 0" rpy="0 0 0" />
+        </inertial>
+      </link>
+      <joint name="navsat_joint" type="revolute">
+        <origin xyz="${-wheelbase/2} 0 0.3" rpy="0 0 0" />
         <parent link="base_link" />
         <child link="navsat_link" />
+        <limit upper="0" lower="0" effort="0" velocity="0" />
       </joint>
+      <!--<joint name="navsat_joint" type="fixed">
+        <origin xyz="${-wheelbase/2} 0 0.3" rpy="0 0 0" />
+        <parent link="base_link" />
+        <child link="navsat_link" />
+      </joint>-->
     </xacro:if>
     <xacro:if value="$(arg velodyne_enabled)">

File: robucar_gazebo/urdf/robucar.gazebo.xacro (robot description, xacro)
@@ -36,10 +36,4 @@
         </plugin>
       </gazebo>
-    </xacro:if>
-    <xacro:if value="$(arg laser_enabled)">
-      <gazebo reference="laser_bracket_link">
-        <material>Gazebo/DarkGrey</material>
-      </gazebo>
-      <xacro:sick_lms100_gazebo prefix="base"/>
     </xacro:if>
     <xacro:if value="$(arg camera_enabled)">
