Commit message: Enable gps frame and use it in gazebo

File: robucar_description/urdf/robucar_4ws.urdf.xacro (robot description, xacro)
@@ -47,5 +47,5 @@
       <link name="navsat_link"/>
       <joint name="navsat_joint" type="fixed">
-        <origin xyz="0.3 0 0.3" rpy="0 0 0" />
+        <origin xyz="${-wheelbase/2} 0 0.3" rpy="0 0 0" />
         <parent link="base_link" />
         <child link="navsat_link" />

File: robucar_description/urdf/wheel_steered.xacro (robot description, xacro)
@@ -34,4 +34,5 @@
       <xacro:insert_block name="joint_origin"/>
       <dynamics damping="0.7"/>
+      <!--<dynamics damping="10.0" friction="20.0" />-->
     </joint>
     <transmission name="${wheel_prefix}_steering_trans" type="SimpleTransmission">

File: robucar_gazebo/urdf/description_4ws.gazebo.xacro (robot description, xacro)
@@ -3,5 +3,5 @@
   <xacro:arg name="laser_enabled" default="false" />
   <xacro:arg name="camera_enabled" default="false" />
-  <xacro:arg name="navsat_enabled" default="false" />
+  <xacro:arg name="navsat_enabled" default="true" />
   <xacro:include filename="$(find robucar_description)/urdf/robucar_4ws.urdf.xacro" />
   <xacro:include filename="$(find robucar_gazebo)/urdf/robucar.gazebo.xacro" />

File: robucar_gazebo/urdf/robucar.gazebo.xacro (robot description, xacro)
@@ -17,21 +17,23 @@
       </plugin>
     </gazebo>
-    <gazebo>
-      <plugin name="gps_controller" filename="libhector_gazebo_ros_gps.so">
-        <updateRate>10</updateRate>
-        <bodyName>base_link</bodyName>
-        <frameId>base_link</frameId>
-        <topicName>navsat/fix</topicName>
-        <velocityTopicName>navsat/vel_simul</velocityTopicName>
-        <referenceLatitude>45.76327</referenceLatitude>
-        <referenceLongitude>3.1094</referenceLongitude>
-        <referenceHeading>0</referenceHeading>
-        <referenceAltitude>400</referenceAltitude>
-        <drift>0.05 0.05 0.05</drift>
-        <gaussianNoise>0.01 0.01 0.01</gaussianNoise>
-        <velocityDrift>0 0 0</velocityDrift>
-        <velocityGaussianNoise>0.01 0.01 0.01</velocityGaussianNoise>
-      </plugin>
-    </gazebo>
+    <xacro:if value="$(arg navsat_enabled)">
+      <gazebo>
+        <plugin name="gps_controller" filename="libhector_gazebo_ros_gps.so">
+          <updateRate>10</updateRate>
+          <bodyName>navsat_link</bodyName>
+          <frameId>navsat_link</frameId>
+          <topicName>navsat/fix</topicName>
+          <velocityTopicName>navsat/vel_simul</velocityTopicName>
+          <referenceLatitude>45.76327</referenceLatitude>
+          <referenceLongitude>3.1094</referenceLongitude>
+          <referenceHeading>0</referenceHeading>
+          <referenceAltitude>400</referenceAltitude>
+          <drift>0.05 0.05 0.05</drift>
+          <gaussianNoise>0.01 0.01 0.01</gaussianNoise>
+          <velocityDrift>0 0 0</velocityDrift>
+          <velocityGaussianNoise>0.01 0.01 0.01</velocityGaussianNoise>
+        </plugin>
+      </gazebo>
+    </xacro:if>
     <xacro:if value="$(arg laser_enabled)">
       <gazebo reference="laser_bracket_link">

Commit message: First working test; but topic latency

File: robucar_description/urdf/robucar_4ws.urdf.xacro (robot description, xacro)
@@ -45,10 +45,22 @@
     </xacro:if>
     <xacro:if value="$(arg navsat_enabled)">
-      <link name="navsat_link"/>
-      <joint name="navsat_joint" type="fixed">
+      <link name="navsat_link">
+        <inertial>
+          <inertia ixx="0.00001" ixy="0.0" ixz="0.0" iyy="0.00001" iyz="0.0" izz="0.00001" />
+          <mass value="0.015" />  <!-- [kg] -->
+          <origin xyz="0 0 0" rpy="0 0 0" />
+        </inertial>
+      </link>
+      <joint name="navsat_joint" type="revolute">
         <origin xyz="${-wheelbase/2} 0 0.3" rpy="0 0 0" />
         <parent link="base_link" />
         <child link="navsat_link" />
+        <limit upper="0" lower="0" effort="0" velocity="0" />
       </joint>
+      <!--<joint name="navsat_joint" type="fixed">
+        <origin xyz="${-wheelbase/2} 0 0.3" rpy="0 0 0" />
+        <parent link="base_link" />
+        <child link="navsat_link" />
+      </joint>-->
     </xacro:if>
     <!--<link name="velodyne"/>

Commit message: Generic vehicle name

File: robucar_description/urdf/robucar_4ws.urdf.xacro (robot description, xacro)
@@ -30,9 +30,10 @@
     </xacro:wheel_steered>
     <xacro:if value="$(arg laser_enabled)">
-      <link name="base_laser"/>
+      <xacro:include filename="$(find lms1xx)/urdf/sick_lms1xx.urdf.xacro"/>
+      <xacro:sick_lms1xx />
       <joint name="laser_joint" type="fixed">
         <origin xyz="${lidar_x_offset} 0.0 ${lidar_ground_clearance - base_z_size/2 - ground_clearance}" rpy="0 0 0" />
         <parent link="base_link" />
-        <child link="base_laser" />
+        <child link="laser" />
       </joint>
     </xacro:if>

Commit message: [description] use 4ws_description pkg

File: robucar_description/urdf/robucar_4ws.urdf.xacro (robot description, xacro)
@@ -1,75 +1,45 @@
 <?xml version="1.0"?>
-<robot name="robucar" xmlns:xacro="http://www.ros.org/wiki/xacro">
+<robot name="robufast" xmlns:xacro="http://www.ros.org/wiki/xacro">
   <xacro:arg name="laser_enabled" default="false" />
   <xacro:arg name="camera_enabled" default="false" />
   <xacro:arg name="navsat_enabled" default="false" />
-  <xacro:include filename="$(find robucar_description)/urdf/wheel_steered.xacro" />
-  <xacro:include filename="$(find robucar_description)/urdf/chassis.xacro" />
-  <xacro:property name="M_PI" value="3.14159"/>
-  <xacro:macro name="robucar">
-    <xacro:chassis/>
-    <!-- IMU Link is the standard mounting position for the IMU.-->
-    <link name="imu_link"/>
-    <joint name="imu_joint" type="fixed">
-      <origin xyz="0.35 0 0.1" rpy="0 0 0" />
-      <parent link="base_link" />
-      <child link="imu_link" />
-    </joint>
-    <!-- Wheel macros -->
-    <xacro:wheel_steered wheel_prefix="front_left" parent_link="base_link" wheel_origin_y="${wheel_y_offset}"  left_right="-1">
-      <origin xyz="${wheelbase/2+wheel_x_offset} ${track/2-wheel_y_offset} ${-base_z_size/2 + wheel_radius - ground_clearance}" rpy="0 0 0" />
-    </xacro:wheel_steered>
-    <xacro:wheel_steered wheel_prefix="front_right" parent_link="base_link" wheel_origin_y="${-wheel_y_offset}"  left_right="1">
-      <origin xyz="${wheelbase/2+wheel_x_offset} ${-track/2+wheel_y_offset} ${-base_z_size/2 + wheel_radius - ground_clearance}" rpy="0 0 0" />
-    </xacro:wheel_steered>
-    <xacro:wheel_steered wheel_prefix="rear_left" parent_link="base_link" wheel_origin_y="${wheel_y_offset}"  left_right="-1">
-      <origin xyz="${-wheelbase/2+wheel_x_offset} ${track/2-wheel_y_offset} ${-base_z_size/2 + wheel_radius - ground_clearance}" rpy="0 0 0" />
-    </xacro:wheel_steered>
-    <xacro:wheel_steered wheel_prefix="rear_right" parent_link="base_link" wheel_origin_y="${-wheel_y_offset}"  left_right="1">
-      <origin xyz="${-wheelbase/2+wheel_x_offset} ${-track/2+wheel_y_offset} ${-base_z_size/2 + wheel_radius - ground_clearance}" rpy="0 0 0" />
-    </xacro:wheel_steered>
-    <xacro:if value="$(arg laser_enabled)">
-      <xacro:include filename="$(find lms1xx)/urdf/sick_lms1xx.urdf.xacro"/>
-      <xacro:sick_lms1xx />
-      <joint name="laser_joint" type="fixed">
-        <origin xyz="${lidar_x_offset} 0.0 ${lidar_ground_clearance - base_z_size/2 - ground_clearance}" rpy="0 0 0" />
-        <parent link="base_link" />
-        <child link="laser" />
-      </joint>
-    </xacro:if>
-    <xacro:if value="$(arg camera_enabled)">
-      <link name="camera_link"/>
-      <joint name="camera_joint" type="fixed">
-        <origin xyz="0.35 0 0.41" rpy="0 0 0" />
-        <parent link="base_link" />
-        <child link="camera_link" />
-      </joint>
-    </xacro:if>
-    <xacro:if value="$(arg navsat_enabled)">
-      <link name="navsat_link">
-        <inertial>
-          <inertia ixx="0.00001" ixy="0.0" ixz="0.0" iyy="0.00001" iyz="0.0" izz="0.00001" />
-          <mass value="0.015" />  <!-- [kg] -->
-          <origin xyz="0 0 0" rpy="0 0 0" />
-        </inertial>
-      </link>
-      <joint name="navsat_joint" type="revolute">
-        <origin xyz="${-wheelbase/2} 0 0.3" rpy="0 0 0" />
-        <parent link="base_link" />
-        <child link="navsat_link" />
-        <limit upper="0" lower="0" effort="0" velocity="0" />
-      </joint>
-      <!--<joint name="navsat_joint" type="fixed">
-        <origin xyz="${-wheelbase/2} 0 0.3" rpy="0 0 0" />
-        <parent link="base_link" />
-        <child link="navsat_link" />
-      </joint>-->
-    </xacro:if>
-    <!--<link name="velodyne"/>
-    <joint name="velodyne_joint" type="fixed">
-      <origin xyz="0.0 0.0 1.0" rpy="0 0 0" />
-      <parent link="base_link" />
-      <child link="velodyne" />
-    </joint>-->
+  <xacro:arg name="velodyne_enabled" default="false" />
+  <xacro:include filename="$(find four_wheel_steering_description)/urdf/chassis.xacro" />
+  <xacro:include filename="$(find four_wheel_steering_description)/urdf/sensors.xacro" />
+  <!-- Base Properties -->
+  <xacro:property name="base_x_size" value="1.66000" />
+  <xacro:property name="base_y_size" value="0.60000" />
+  <xacro:property name="base_z_size" value="0.66000" />
+  <xacro:property name="wheelbase" value="1.2" />
+  <xacro:property name="track" value="1.1" />
+  <xacro:property name="mass_base" value="500" />
+  <!-- Wheel Properties -->
+  <xacro:property name="steering_link_mass" value="30" />
+  <xacro:property name="mass_wheel" value="5" />
+  <xacro:property name="wheel_length" value="0.2" />
+  <xacro:property name="wheel_radius" value="0.45" />
+  <!-- Wheel Mounting Positions -->
+  <xacro:property name="ground_clearance" value="0.35" />
+  <xacro:property name="wheel_x_offset" value="0.0" />
+  <xacro:property name="wheel_y_offset" value="0.1" />
+  <!-- LIDAR Properties -->
+  <xacro:property name="lidar_ground_clearance" value="0.69" />
+  <xacro:property name="lidar_x_offset" value="1.2" />
+  <xacro:macro name="robufast">
+    <xacro:chassis>
+      <!-- visual chassis -->
+      <visual>
+        <origin xyz="0.03 0 ${-base_z_size/2}" rpy="0 0 ${M_PI/2.0}" />
+        <geometry>
+          <mesh filename="package://robucar_description/meshes/chassis.dae"/>
+        </geometry>
+      </visual>
+      <!-- visual steering -->
+      <mesh filename="package://robucar_description/meshes/wheel_steered.dae"/>
+      <!-- visual wheel -->
+      <mesh filename="package://robucar_description/meshes/wheel.dae"/>
+    </xacro:chassis>
+    <xacro:sensors/>
   </xacro:macro>
+  <xacro:robufast />
 </robot>

Commit message: [description] Update meshe files

File: robucar_description/urdf/robucar_4ws.urdf.xacro (robot description, xacro)
@@ -11,14 +11,14 @@
   <xacro:property name="base_y_size" value="0.60000" />
   <xacro:property name="base_z_size" value="0.66000" />
-  <xacro:property name="wheelbase" value="1.2" />
-  <xacro:property name="track" value="1.1" />
-  <xacro:property name="mass_base" value="500" />
+  <xacro:property name="wheelbase" value="1.22" />
+  <xacro:property name="track" value="1.23" />
+  <xacro:property name="mass_base" value="340" />
   <!-- Wheel Properties -->
   <xacro:property name="steering_link_mass" value="30" />
   <xacro:property name="mass_wheel" value="5" />
-  <xacro:property name="wheel_length" value="0.2" />
-  <xacro:property name="wheel_radius" value="0.45" />
+  <xacro:property name="wheel_length" value="0.1" />
+  <xacro:property name="wheel_radius" value="0.28" />
   <!-- Wheel Mounting Positions -->
-  <xacro:property name="ground_clearance" value="0.35" />
+  <xacro:property name="ground_clearance" value="0.19" />
   <xacro:property name="wheel_x_offset" value="0.0" />
   <xacro:property name="wheel_y_offset" value="0.1" />
@@ -30,5 +30,5 @@
       <!-- visual chassis -->
       <visual>
-        <origin xyz="0.03 0 ${-base_z_size/2}" rpy="0 0 ${M_PI/2.0}" />
+        <origin xyz="0 0 ${-base_z_size/2}" rpy="0 0 ${M_PI/2.0}" />
         <geometry>
           <mesh filename="package://robucar_description/meshes/chassis.dae"/>
